Commit message: update myAGV.urdf

File: myagv_description/urdf/myAGV.urdf (robot description, URDF)
Before this commit: robot myAGV, 2 links, 1 joints
Joints:
- joint base_joint: child base_up -> base_link

Commit message: update myAGV.urdf

File: myagv_description/urdf/myAGV.urdf (robot description, URDF)
Before this commit: robot myAGV, 2 links, 1 joints
Links:
- link base_footprint: geometry visual mesh filename=package://myagv_description/meshes/myagv_base.dae scale=1 1 1
- link base_link: geometry visual mesh filename=package://myagv_description/meshes/myagv_up.dae scale=1 1 1
